Commit message: ready the simmulation for AI trainning

File: src/torto_description/urdf/torto.urdf (robot description, URDF)
Before this commit: robot TORTO, 13 links, 12 joints
Links:
- added link tortoIMU_link; visual mesh filename=package://torto_description/meshes/sensors/torto_MPU6050.stl scale=0.001 0.001 0.001
- added link tortoLidar_link; visual mesh filename=package://torto_description/meshes/sensors/torto_YDLidarX3.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 scale=0.001 0.001 0.001
- link tortoTiBiaBL_link: mass 3.29 -> 0.07
Joints:
- added joint body_tortoIMU_joint: type fixed, parent tortoBody_link, child tortoIMU_link, origin xyz=-0.0676 -0.03725 0.00062 rpy=0 0 0, axis 0 0 0
- added joint body_tortoLidar_joint: type fixed, parent tortoBody_link, child tortoLidar_link, origin xyz=0.037 0 0.1282 rpy=0 0 0, axis 0 0 0
- joint FemurBL_TiBiaBL_joint: axis 1 0 0 -> 0 1 0; origin xyz=0 -0.09 0 rpy=0 0 0 -> xyz=0.09 0 0 rpy=0 0 0
- joint FemurBR_TiBiaBR_joint: axis 1 0 0 -> 0 1 0; origin xyz=0 -0.09 0 rpy=0 0 0 -> xyz=0.09 0 0 rpy=0 0 0
- joint FemurFL_TiBiaFL_joint: axis 1 0 0 -> 0 1 0; origin xyz=0 0.09 0 rpy=0 0 0 -> xyz=-0.09 0 0 rpy=0 0 0
- joint FemurFR_TiBiaFR_joint: axis 1 0 0 -> 0 1 0; origin xyz=0 0.09 0 rpy=0 0 0 -> xyz=-0.09 0 0 rpy=0 0 0
- joint body_detoidBL_joint: axis 0 1 0 -> -1 0 0; origin xyz=0.07 0.0876 -0.0143 rpy=0 0 0 -> xyz=-0.0876 0.07 -0.0143 rpy=0 0 0
- joint body_detoidBR_joint: axis 0 1 0 -> -1 0 0; origin xyz=-0.07 0.0876 -0.0143 rpy=0 0 0 -> xyz=-0.0876 -0.07 -0.0143 rpy=0 0 0
- joint body_detoidFL_joint: axis 0 1 0 -> -1 0 0; origin xyz=0.07 -0.0876 -0.0143 rpy=0 0 0 -> xyz=0.0876 0.07 -0.0143 rpy=0 0 0
- joint body_detoidFR_joint: axis 0 1 0 -> -1 0 0; origin xyz=-0.07 -0.0876 -0.0143 rpy=0 0 0 -> xyz=0.0876 -0.07 -0.0143 rpy=0 0 0
- joint detoidBL_FemurBL_joint: axis 1 0 0 -> 0 1 0; origin xyz=0.0406 0.050152 -0.012844 rpy=0 0 0 -> xyz=-0.050152 0.0406 -0.012844 rpy=0 0 0
- joint detoidBR_FemurBR_joint: axis 1 0 0 -> 0 1 0; origin xyz=-0.0406 0.050152 -0.012844 rpy=0 0 0 -> xyz=-0.050152 -0.0406 -0.012844 rpy=0 0 0
- joint detoidFL_FemurFL_joint: axis 1 0 0 -> 0 1 0; origin xyz=0.0406 -0.050152 -0.012844 rpy=0 0 0 -> xyz=0.050152 0.0406 -0.012844 rpy=0 0 0
- joint detoidFR_FemurFR_joint: axis 1 0 0 -> 0 1 0; origin xyz=-0.0406 -0.050152 -0.012844 rpy=0 0 0 -> xyz=0.050152 -0.0406 -0.012844 rpy=0 0 0
